File: hardware/secondary/companion.brd (EAGLE design)
At the start: 32 x 28.1 mm, 13 parts, among them U1 USD-SOCKET

Commit message: New hardware revision, better connector.
Parts:
- added C1: (no value), SparkFun-Capacitors:0805
- added JP2: (no value), SparkFun-Connectors:1X04_LOCK
- added U$11, U$12: 1.27MM-MILLMAX, 1.27mm-headers:1X03-1.27MM
Connections:
- new net GND_DB: JP2.4, U$12.4
- new net RX1: JP2.2, U$12.2
- new net TX0: JP2.3, U$12.3
- new net VCC_DB: JP2.1, U$12.1
- net GND: now also C1.2, U$11.4
- net SD_CLK: now also U$11.1
- net SD_SIMO: now also U$11.3
- net SD_SOMI: now also U$11.2
- net SD_VCC: now also C1.1
Routing:
- net SD_SOMI: track 15.7 -> 25.3 mm
- net VCC_DB: track 0.00 -> 6.56 mm
- net RX1: track 0.00 -> 6.29 mm
- net TX0: track 0.00 -> 6.04 mm
- net SD_VCC: track 19.9 -> 24.5 mm
- net SD_SIMO: track 16.5 -> 21.1 mm, vias 1 -> 2
- net SD_CLK: track 14.5 -> 17.4 mm
- added copper zone on layer 1, net GND_DB
Other:
- outline, holes or cut-outs redrawn
- board text added: "<SPI / UART Debug>"
- board text added: "Amulet "Kite" Rev. G Storage Board"
- board text added: "Amulet "Snail Kite" BLE Debug Board"
- board text added: "CLK"
- board text added: "DNP"
- board text added: "RX"
- board text added: "TX"
- board text added: "VCC"
- board text removed: "Amulet "Snail Kite" Rev. G Storage Board"
