File: hardware/secondary/companion.sch (EAGLE design)
At the start: 13 parts, among them U1 USD-SOCKET

Commit message: New hardware revision, better connector.
Parts:
- added C1: (no value), SparkFun-Capacitors:CAP0805
- added JP2: (no value), SparkFun-Connectors:M04LOCK
- added U$11, U$12: 1.27MM-MILLMAX, 1.27mm-headers:1.27MM-MILLMAX
- JP3: DIGIKEY (none) -> H11622CT-ND
Connections:
- new net GND_DB: JP2.4, U$12.4
- new net RX1: JP2.2, U$12.2
- new net TX0: JP2.3, U$12.3
- new net VCC_DB: JP2.1, U$12.1
- net GND: now also C1.2, U$11.4
- net SD_CLK: now also U$11.1
- net SD_SIMO: now also U$11.3
- net SD_SOMI: now also U$11.2
- net SD_VCC: now also C1.1
Other:
- note added: "BLE Debug Board"
- note added: "RX"
- note added: "TX"
- note removed: "Copyright 2016 by the Trustees of Dartmouth College and Clemson University, and distributed under the terms of the "Dartmouth College Non-Exclusive Research Use Source Code License Agreement" (for NON-COMMERCIAL research purposes only), as detailed in a file named LICENSE.pdf within this repository."
- note removed: "LICENSE"
- moved on the sheet: JP1
