File: hardware/watch/watch.sch (EAGLE design)
At the start: 92 parts, among them IC1 Digikey: WM9203CT-ND, IC2 MPR121, Q1 NTS4173, Q3 NTS4173, Q4 NTS4173, U1 Value, U10 2450BM14E0003, U11 MCP73831, U12 ML8511-UV-SENSORSMD, U13 LIGHTSENSORALS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

Commit message: Added license text to remaining files, and to CAD EAGLE schematics.
Other:
- note added: "Copyright 2016 by the Trustees of Dartmouth College and Clemson University, and distributed under the terms of the "Dartmouth College Non-Exclusive Research Use Source Code License Agreement" (for NON-COMMERCIAL research purposes only), as detailed in a file named LICENSE.pdf within this repository."
- note added: "LICENSE"
Changed lines of the file:
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@@
 When USB plugged, BATT disconnect from U9</text>
 <text x="35.56" y="200.66" size="5.08" layer="97">MSP430 Prog</text>
+<text x="7.62" y="7.62" size="3.302" layer="97" font="vector" ratio="15">Copyright 2016 by the Trustees of Dartmouth College
+and Clemson University, and distributed under the terms
+of the "Dartmouth College Non-Exclusive Research Use
+Source Code License Agreement" (for NON-COMMERCIAL
+research purposes only), as detailed in a file named
+LICENSE.pdf within this repository.</text>
+<text x="7.62" y="38.1" size="5.08" layer="97" font="vector" ratio="23">LICENSE</text>
+<wire x1="7.62" y1="48.26" x2="167.64" y2="48.26" width="1.27" layer="97" style="longdash"/>
+<wire x1="167.64" y1="48.26" x2="167.64" y2="2.54" width="1.27" layer="97" style="longdash"/>
 </plain>
 <instances>

Commit message: New hardware revision, better connector.
Parts:
- removed C27: 2.2uF, tiny_passives:C-EU
- removed D4: BAT20J, SparkFun-DiscreteSemi:DIODE-SCHOTTKY-BAT20J
- removed Q4: NTS4173, nts4173p:NTS4173
- removed R4: 220k, tiny_passives:R-EU
- added JP2: (no value), SparkFun-Connectors:M041.27MM
- renumbered U$1 to JP3
Connections:
- removed net !GYRO_ENABLE: U1.P1.4_UCB0CLK_UCA0STE_TA1.0
- removed net V_PRE_REG: C27.2, D4.C, Q4.S, U9.CE, U9.VIN
- new net DEBUG_BLE_RX: JP2.3, U4.P18
- new net DEBUG_BLE_TX: JP2.4, U4.P17
- net GND: now also JP2.1; no longer C27.1, R4.1
- net V+: now also JP2.2
- net VBAT: now also U9.CE, U9.VIN; no longer Q4.D
- net VIN: no longer D4.A, Q4.G, R4.2
Other:
- note added: "INMP510"
- note added: "P15-P16 connect to VDD P9-P13 connecto GND"
- note removed: "Copyright 2016 by the Trustees of Dartmouth College and Clemson University, and distributed under the terms of the "Dartmouth College Non-Exclusive Research Use Source Code License Agreement" (for NON-COMMERCIAL research purposes only), as detailed in a file named LICENSE.pdf within this repository."
- note removed: "LICENSE"
- note removed: "Load Sharing: P-FET pulled to GND when no USB plug which allows current from BATT to U9 When USB plugged, BATT disconnect from U9"
